File: wissystem_beatseq1/wissystem_beatseq1.kicad_pcb (KiCad board)
At the start: 2 copper layers, 20.3 x 128.5 mm, 46 parts, among them J1 EuroPower16, J2 Thonkiconn, J3 Thonkiconn, Q1 NPN S8050 J3Y, Q2 NPN S8050 J3Y, Q3 NPN S8050 J3Y, Q4 NPN S8050 J3Y, Q5 NPN S8050 J3Y, SW1 SW_SPST, SW2 SW_SPST, SW3 SW_SPST, SW4 SW_SPST, U1 TL072CDT, U2 CD4017BM, U3 TL072CDT, U4 TL072CDT

Commit message: made protoboard for the latching switches
Parts:
- removed C1, C2, C3, C4: 10u, kpm-jlcpcb-basic:C_0402_1005Metric
- removed J2, J3: Thonkiconn, EuroRackTools:Jack_3.5mm_QingPu_WQP-PJ398SM_Vertical_CircularHoles
- removed Q1, Q2, Q3, Q4, Q5: NPN S8050 J3Y, kpm-jlcpcb-basic:SOT-23
- removed R1: 1k, kpm-jlcpcb-basic:R_0603_1608Metric
- removed R15, R16, R17, R18: 100k, kpm-jlcpcb-basic:R_0402_1005Metric
- added D10: blue, kpm-jlcpcb-basic:LED_0603_1608Metric, F.Cu at (25.6, 86.1)
- added D11: 1N4148WS, EuroRackTools:D_SOD-323, F.Cu at (30.1, 94.8)
- added D12: blue, kpm-jlcpcb-basic:LED_0603_1608Metric, F.Cu at (25.6, 94.5)
- added D13: 1N4148WS, EuroRackTools:D_SOD-323, F.Cu at (30.1, 103.2)
- added D14: blue, kpm-jlcpcb-basic:LED_0603_1608Metric, F.Cu at (25.6, 103.0)
- added D15: 1N4148WS, EuroRackTools:D_SOD-323, F.Cu at (30.3, 111.6)
- added D16: blue, kpm-jlcpcb-basic:LED_0603_1608Metric, F.Cu at (25.6, 111.4)
- added D17: 1N4148WS, EuroRackTools:D_SOD-323, F.Cu at (27.7, 114.4)
- added D18: 1N4148WS, EuroRackTools:D_SOD-323, F.Cu at (22.5, 114.4)
- added D9: 1N4148WS, EuroRackTools:D_SOD-323, F.Cu at (30.1, 86.4)
- added J10: Conn_01x05, Connector_PinSocket_2.54mm:PinSocket_1x05_P2.54mm_Vertical, F.Cu at (61.3, 109.0)
- added J11: Conn_01x03, Connector_PinSocket_2.54mm:PinSocket_1x03_P2.54mm_Vertical, F.Cu at (47.9, 92.5)
- added J12: Conn_01x05, Connector_PinSocket_2.54mm:PinSocket_1x05_P2.54mm_Vertical, F.Cu at (61.3, 95.3)
- added J13: Conn_01x03, Connector_PinSocket_2.54mm:PinSocket_1x03_P2.54mm_Vertical, F.Cu at (47.9, 78.8)
- added J14: Conn_01x05, Connector_PinSocket_2.54mm:PinSocket_1x05_P2.54mm_Vertical, F.Cu at (61.3, 81.6)
- added J15: Conn_01x03, Connector_PinSocket_2.54mm:PinSocket_1x03_P2.54mm_Vertical, F.Cu at (47.9, 65.1)
- added J16: Conn_01x05, Connector_PinSocket_2.54mm:PinSocket_1x05_P2.54mm_Vertical, F.Cu at (61.3, 67.9)
- added J17: Conn_01x03, Connector_PinSocket_2.54mm:PinSocket_1x03_P2.54mm_Vertical, F.Cu at (47.9, 51.4)
- added J18: Conn_01x05, Connector_PinSocket_2.54mm:PinSocket_1x05_P2.54mm_Vertical, F.Cu at (61.3, 54.2)
- added J19: Conn_01x03, Connector_PinSocket_2.54mm:PinSocket_1x03_P2.54mm_Vertical, F.Cu at (47.9, 37.7)
- added J20: Conn_01x05, Connector_PinSocket_2.54mm:PinSocket_1x05_P2.54mm_Vertical, F.Cu at (61.3, 40.5)
- added J21: Conn_01x02, Connector_PinSocket_2.54mm:PinSocket_1x02_P2.54mm_Vertical, F.Cu at (35.8, 80.0)
- added J22: Conn_01x02, Connector_PinSocket_2.54mm:PinSocket_1x02_P2.54mm_Vertical, F.Cu at (34.4, 89.6)
- added J4: Conn_01x03, Connector_PinSocket_2.54mm:PinSocket_1x03_P2.54mm_Vertical, F.Cu at (34.8, 75.3)
- added J5: Conn_01x03, Connector_PinSocket_2.54mm:PinSocket_1x03_P2.54mm_Vertical, F.Cu at (47.9, 133.6)
- added J6: Conn_01x05, Connector_PinSocket_2.54mm:PinSocket_1x05_P2.54mm_Vertical, F.Cu at (61.3, 136.4)
- added J7: Conn_01x03, Connector_PinSocket_2.54mm:PinSocket_1x03_P2.54mm_Vertical, F.Cu at (47.9, 119.9)
- added J8: Conn_01x05, Connector_PinSocket_2.54mm:PinSocket_1x05_P2.54mm_Vertical, F.Cu at (61.3, 122.7)
- added J9: Conn_01x03, Connector_PinSocket_2.54mm:PinSocket_1x03_P2.54mm_Vertical, F.Cu at (47.9, 106.2)
- added JCLK1: Thonkiconn, EuroRackTools:Jack_3.5mm_QingPu_WQP-PJ398SM_Vertical_CircularHoles, F.Cu at (35.7, 135.6)
- added JCLK2: Thonkiconn, EuroRackTools:Jack_3.5mm_QingPu_WQP-PJ398SM_Vertical_CircularHoles, F.Cu at (37.1, 115.2)
- added JDEC1: Conn_01x01, Connector_PinSocket_2.54mm:PinSocket_1x01_P2.54mm_Vertical, F.Cu at (54.7, 30.7)
- added JDEC10: Conn_01x01, Connector_PinSocket_2.54mm:PinSocket_1x01_P2.54mm_Vertical, F.Cu at (43.9, 95.1)
- added JDEC11: Conn_01x01, Connector_PinSocket_2.54mm:PinSocket_1x01_P2.54mm_Vertical, F.Cu at (43.9, 54.0)
- added JDEC12: Conn_01x01, Connector_PinSocket_2.54mm:PinSocket_1x01_P2.54mm_Vertical, F.Cu at (43.9, 108.8)
- added JDEC13: Conn_01x01, Connector_PinSocket_2.54mm:PinSocket_1x01_P2.54mm_Vertical, F.Cu at (43.9, 67.7)
- added JDEC14: Conn_01x01, Connector_PinSocket_2.54mm:PinSocket_1x01_P2.54mm_Vertical, F.Cu at (43.9, 122.5)
- added JDEC15: Conn_01x01, Connector_PinSocket_2.54mm:PinSocket_1x01_P2.54mm_Vertical, F.Cu at (43.9, 81.4)
- added JDEC16: Conn_01x01, Connector_PinSocket_2.54mm:PinSocket_1x01_P2.54mm_Vertical, F.Cu at (43.9, 136.2)
- added JDEC17: Conn_01x01, Connector_PinSocket_2.54mm:PinSocket_1x01_P2.54mm_Vertical, F.Cu at (34.3, 100.2)
- added JDEC18: Conn_01x01, Connector_PinSocket_2.54mm:PinSocket_1x01_P2.54mm_Vertical, F.Cu at (37.2, 86.5)
- added JDEC19: Conn_01x01, Connector_PinSocket_2.54mm:PinSocket_1x01_P2.54mm_Vertical, F.Cu at (34.3, 96.5)
- added JDEC2: Conn_01x01, Connector_PinSocket_2.54mm:PinSocket_1x01_P2.54mm_Vertical, F.Cu at (55.0, 44.3)
- added JDEC20: Conn_01x01, Connector_PinSocket_2.54mm:PinSocket_1x01_P2.54mm_Vertical, F.Cu at (41.4, 85.1)
- added JDEC21: Conn_01x01, Connector_PinSocket_2.54mm:PinSocket_1x01_P2.54mm_Vertical, F.Cu at (33.4, 84.4)
- added JDEC3: Conn_01x01, Connector_PinSocket_2.54mm:PinSocket_1x01_P2.54mm_Vertical, F.Cu at (55.0, 57.9)
- added JDEC4: Conn_01x01, Connector_PinSocket_2.54mm:PinSocket_1x01_P2.54mm_Vertical, F.Cu at (55.0, 71.4)
- added JDEC5: Conn_01x01, Connector_PinSocket_2.54mm:PinSocket_1x01_P2.54mm_Vertical, F.Cu at (54.9, 85.0)
- added JDEC6: Conn_01x01, Connector_PinSocket_2.54mm:PinSocket_1x01_P2.54mm_Vertical, F.Cu at (54.9, 98.5)
- added JDEC7: Conn_01x01, Connector_PinSocket_2.54mm:PinSocket_1x01_P2.54mm_Vertical, F.Cu at (54.9, 112.1)
- added JDEC8: Conn_01x01, Connector_PinSocket_2.54mm:PinSocket_1x01_P2.54mm_Vertical, F.Cu at (54.9, 125.7)
- added JDEC9: Conn_01x01, Connector_PinSocket_2.54mm:PinSocket_1x01_P2.54mm_Vertical, F.Cu at (43.9, 40.3)
- added JOUT1: Thonkiconn, EuroRackTools:Jack_3.5mm_QingPu_WQP-PJ398SM_Vertical_CircularHoles, F.Cu at (25.7, 135.6)
- added SW41: PUSHBTN_DPDT_LATCH, EuroRackTools:SMD switch 6pin, F.Cu at (54.6, 131.2)
- added SW42: PUSHBTN_DPDT_LATCH, EuroRackTools:SMD switch 6pin, F.Cu at (54.6, 117.5)
- added SW43: PUSHBTN_DPDT_LATCH, EuroRackTools:SMD switch 6pin, F.Cu at (54.6, 90.1)
- added SW44: PUSHBTN_DPDT_LATCH, EuroRackTools:SMD switch 6pin, F.Cu at (54.6, 103.8)
- added SW45: PUSHBTN_DPDT_LATCH, EuroRackTools:SMD switch 6pin, F.Cu at (54.6, 76.4)
- added SW46: PUSHBTN_DPDT_LATCH, EuroRackTools:SMD switch 6pin, F.Cu at (54.6, 62.7)
- added SW47: PUSHBTN_DPDT_LATCH, EuroRackTools:SMD switch 6pin, F.Cu at (54.6, 49.0)
- added SW48: PUSHBTN_DPDT_LATCH, EuroRackTools:SMD switch 6pin, F.Cu at (54.6, 35.3)
- added SW5: PUSHBTN_DPDT_LATCH, EuroRackTools:SMD switch 6pin, F.Cu at (25.8, 82.2)
- added SW6: PUSHBTN_DPDT_LATCH, EuroRackTools:SMD switch 6pin, F.Cu at (25.8, 90.6)
- added SW7: PUSHBTN_DPDT_LATCH, EuroRackTools:SMD switch 6pin, F.Cu at (25.8, 99.0)
- added SW8: PUSHBTN_DPDT_LATCH, EuroRackTools:SMD switch 6pin, F.Cu at (25.8, 107.4)
- added U12: CD4017BM, EuroRackTools:SOP-16_4.4x10.4mm_P1.27mm, F.Cu at (37.5, 63.6)
- D1, D6: value red -> blue
- D3, D5: value red -> 1N4148WS; footprint kpm-jlcpcb-basic:LED_0603_1608Metric -> EuroRackTools:D_SOD-323
- D4, D8: value 1N4148WS -> blue; footprint EuroRackTools:D_SOD-323 -> kpm-jlcpcb-basic:LED_0603_1608Metric
- R10, R11, R6, R7: value 1.2k -> 4.7k
- R12, R14: value 1.2k -> 100k
- R13: value 100k -> 1k; footprint kpm-jlcpcb-basic:R_0402_1005Metric -> kpm-jlcpcb-basic:R_0603_1608Metric
- R2, R3: value 1.2k -> 150k
- R4, R5, R8, R9: value 100k -> 4.7k
- SW1, SW2, SW3, SW4: value SW_SPST -> PUSHBTN_DPDT_LATCH; footprint EuroRackTools:SW_SPST_PTS645 -> EuroRackTools:SMD switch 6pin
- moved R2 88.1 mm to (31.2, 118.6), turned to -90 degrees
- moved R3 85.0 mm to (31.2, 120.5)
- moved J1 80.4 mm to (38.2, 34.8)
- moved U3 80.1 mm to (25.1, 118.1), turned to 90 degrees
- moved R13 72.7 mm to (22.1, 121.8), turned to 180 degrees
- moved R12 65.1 mm to (25.1, 114.9), turned to 0 degrees
- moved U2 62.7 mm to (25.8, 40.0), turned to 0 degrees
- moved R14 58.0 mm to (21.0, 116.3), turned to -90 degrees
- moved R11 57.8 mm to (23.1, 111.2), turned to 180 degrees
- moved R10 57.1 mm to (23.1, 102.8), turned to 180 degrees
- moved R9 55.4 mm to (23.1, 94.4), turned to 180 degrees
- moved R8 49.7 mm to (23.1, 86.0), turned to 180 degrees
- moved U4 44.5 mm to (39.4, 98.1), turned to 0 degrees
- moved R7 41.5 mm to (23.1, 77.6), turned to 180 degrees
- moved R5 34.1 mm to (23.1, 60.8)
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Connections:
- D2 pad 1: Net-(D2-K) -> Net-(D11-K)
- D3 pad 1: Net-(D3-K) -> Net-(D11-K)
- D4 pad 1: Net-(D2-K) -> Net-(D4-K)
- D5 pad 1: Net-(D5-K) -> Net-(D11-K)
- D7 pad 1: Net-(D2-K) -> Net-(D11-K)
- D8 pad 1: Net-(D2-K) -> Net-(D8-K)
- R10 pad 1: Net-(SW3-A) -> Net-(D14-K)
- R10 pad 2: Net-(R10-Pad2) -> GND
- R11 pad 1: Net-(SW4-A) -> Net-(D16-K)
- R11 pad 2: Net-(R11-Pad2) -> GND
- R12 pad 1: Net-(D5-A) -> Net-(R12-Pad1)
- R12 pad 2: Net-(R10-Pad2) -> Net-(D17-A)
- R13 pad 1: GND -> Net-(U3B--)
- R13 pad 2: Net-(D5-A) -> Net-(JOUT1-PadT)
- R14 pad 1: Net-(D6-A) -> Net-(D18-K)
- R14 pad 2: Net-(R11-Pad2) -> GND
- R2 pad 1: Net-(SW1-A) -> +5V
- R3 pad 1: Net-(D1-A) -> Net-(R2-Pad2)
- R3 pad 2: Net-(R2-Pad2) -> GND
- R4 pad 1: GND -> Net-(D1-K)
- R4 pad 2: Net-(D1-A) -> GND
- R5 pad 1: GND -> Net-(D4-K)
- R5 pad 2: Net-(D2-A) -> GND
- R6 pad 1: Net-(SW2-A) -> Net-(D6-K)
- R6 pad 2: Net-(R6-Pad2) -> GND
- R7 pad 1: Net-(D3-A) -> Net-(D8-K)
- R7 pad 2: Net-(R6-Pad2) -> GND
- R8 pad 1: GND -> Net-(D10-K)
- R8 pad 2: Net-(D3-A) -> GND
- R9 pad 1: GND -> Net-(D12-K)
- R9 pad 2: Net-(D4-A) -> GND
- SW1 pad 1: Net-(SW1-A) -> unconnected-(SW1-A-Pad1)
- SW1 pad 2: Net-(SW1-B) -> Net-(U2-Q0)
- SW2 pad 1: Net-(SW2-A) -> unconnected-(SW2-A-Pad1)
- SW2 pad 2: Net-(SW2-B) -> Net-(U2-Q1)
- SW3 pad 1: Net-(SW3-A) -> unconnected-(SW3-A-Pad1)
- SW3 pad 2: Net-(SW3-B) -> Net-(U2-Q2)
- SW4 pad 1: Net-(SW4-A) -> unconnected-(SW4-A-Pad1)
- SW4 pad 2: Net-(SW4-B) -> Net-(U2-Q3)
- U1 pad 2: clock -> ref
- U2 pad 1: beat6 -> Net-(U2-Q5)
- U2 pad 10: beat5 -> Net-(U2-Q4)
- U2 pad 15: unconnected-(U2-Reset-Pad15) -> Net-(U2-Q8)
- U2 pad 16: +12V -> +5V
- U2 pad 2: beat2 -> Net-(U2-Q1)
- U2 pad 3: beat1 -> Net-(U2-Q0)
- U2 pad 4: beat3 -> Net-(U2-Q2)
- U2 pad 5: beat7 -> Net-(U2-Q6)
- U2 pad 6: beat8 -> Net-(U2-Q7)
- U2 pad 7: beat4 -> Net-(U2-Q3)
- U2 pad 9: unconnected-(U2-Q8-Pad9) -> Net-(U2-Q8)
- U3 pad 1: Net-(R2-Pad2) -> Net-(R12-Pad1)
- U3 pad 2: Net-(SW1-B) -> ref
- U3 pad 3: Net-(D1-A) -> Net-(D11-K)
- U3 pad 5: Net-(D3-A) -> Net-(D18-K)
- U3 pad 6: Net-(SW2-B) -> Net-(U3B--)
- U3 pad 7: Net-(R6-Pad2) -> Net-(U3B--)
- U4 pad 1: Net-(R10-Pad2) -> Net-(JDEC18-Pin_1)
- U4 pad 2: Net-(SW3-B) -> Net-(J21-Pin_1)
- U4 pad 3: Net-(D5-A) -> Net-(J21-Pin_2)
- U4 pad 5: Net-(D6-A) -> Net-(J22-Pin_2)
- U4 pad 6: Net-(SW4-B) -> Net-(J22-Pin_1)
- U4 pad 7: Net-(R11-Pad2) -> Net-(JDEC19-Pin_1)
Routing:
- net +5V: track 2.54 -> 283.8 mm, vias 0 -> 3
- net clock: track 12.0 -> 126.2 mm, vias 0 -> 2
- net Net-(J4-Pin_3): track 0.00 -> 100.1 mm
- net ref: track 0.00 -> 87.9 mm, vias 0 -> 2
- net beat1: track 85.6 -> 0.00 mm
- net beat3: track 82.2 -> 0.00 mm, vias 2 -> 0
- net Net-(D2-K): track 79.0 -> 0.00 mm, vias 3 -> 0
- net Net-(JDEC8-Pin_1): track 0.00 -> 75.2 mm, vias 0 -> 2
- net beat2: track 72.6 -> 0.00 mm
- net Net-(D11-K): track 0.00 -> 66.8 mm
- net Net-(U2-Q7): track 0.00 -> 65.2 mm, vias 0 -> 2
- net Net-(JDEC7-Pin_1): track 0.00 -> 61.1 mm, vias 0 -> 2
- net Net-(D7-A): track 61.7 -> 2.21 mm, vias 2 -> 0
- net Net-(U2-Q6): track 0.00 -> 58.1 mm, vias 0 -> 2
- net beat4: track 52.8 -> 0.00 mm
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Other:
- board size 20.3 x 128.5 mm -> 45.7 x 128.5 mm
- board text added: "+"
- board text added: "1"
- board text added: "2"
- board text added: "3"
- board text added: "4"
- board text added: "5"
- board text added: "6"
- board text added: "CLK"
- board text added: "COM"
- board text added: "G"
- board text added: "REF"
- board text added: "wis designs 2023"
