File: wissystem_beatseq1/wissystem_beatseq1.kicad_sch (KiCad schematic)
At the start: 46 parts, among them J1 EuroPower16, J2 Thonkiconn, J3 Thonkiconn, Q1 NPN S8050 J3Y, Q2 NPN S8050 J3Y, Q3 NPN S8050 J3Y, Q4 NPN S8050 J3Y, Q5 NPN S8050 J3Y, SW1 SW_SPST, SW2 SW_SPST, SW3 SW_SPST, SW4 SW_SPST, U1 TL072CDT, U2 CD4017BM, U3 TL072CDT, U4 TL072CDT

Commit message: made protoboard for the latching switches
Parts:
- removed C1, C2, C3, C4: 10u, kpm-jlcpcb-basic:C_0402_1005Metric, symbol kpm-jlcpcb-basic:10u C 0402
- removed D1, D3, D5, D6: red, kpm-jlcpcb-basic:LED_0603_1608Metric, symbol kpm-jlcpcb-basic:red LED 0603
- removed D4, D8: 1N4148WS, EuroRackTools:D_SOD-323, symbol EuroRackTools:1N4148WS
- removed J3: Thonkiconn, EuroRackTools:Jack_3.5mm_QingPu_WQP-PJ398SM_Vertical_CircularHoles, symbol EuroRackTools:Thonkiconn
- removed Q1, Q2, Q3, Q4, Q5: NPN S8050 J3Y, kpm-jlcpcb-basic:SOT-23, symbol kpm-jlcpcb-basic:NPN S8050 J3Y
- removed R1: 1k, kpm-jlcpcb-basic:R_0603_1608Metric, symbol kpm-jlcpcb-basic:1k R 0603
- removed R10, R11, R12, R14, R2, R3, R6, R7: 1.2k, kpm-jlcpcb-basic:R_0402_1005Metric, symbol kpm-jlcpcb-basic:1.2k R 0402
- removed R13, R15, R16, R17, R18, R4, R5, R8, R9: 100k, kpm-jlcpcb-basic:R_0402_1005Metric, symbol kpm-jlcpcb-basic:100k R 0402
- removed SW1, SW2, SW3, SW4: SW_SPST, EuroRackTools:SW_SPST_PTS645, symbol EuroRackTools:PUSHBTN
- added D1, D10, D12, D14, D16, D4, D6, D8: blue, kpm-jlcpcb-basic:LED_0603_1608Metric, symbol kpm-jlcpcb-basic:blue LED 0603
- added D11, D13, D15, D17, D18, D3, D5, D9: 1N4148WS, EuroRackTools:D_SOD-323, symbol EuroRackTools:1N4148WS
- added J10, J12, J14, J16, J18, J20, J6, J8: Conn_01x05, Connector_PinSocket_2.54mm:PinSocket_1x05_P2.54mm_Vertical, symbol Connector_Generic:Conn_01x05
- added J11, J13, J15, J17, J19, J4, J5, J7, J9: Conn_01x03, Connector_PinSocket_2.54mm:PinSocket_1x03_P2.54mm_Vertical, symbol Connector_Generic:Conn_01x03
- added J2, J3: Conn_01x01, symbol Connector_Generic:Conn_01x01
- added J21, J22: Conn_01x02, Connector_PinSocket_2.54mm:PinSocket_1x02_P2.54mm_Vertical, symbol Connector_Generic:Conn_01x02
- added JCLK2, JOUT1: Thonkiconn, EuroRackTools:Jack_3.5mm_QingPu_WQP-PJ398SM_Vertical_CircularHoles, symbol EuroRackTools:Thonkiconn
- added JDEC1, JDEC10, JDEC11, JDEC12, JDEC13, JDEC14, JDEC15, JDEC16, JDEC17, JDEC18, JDEC19, JDEC2, JDEC20, JDEC21, JDEC3, JDEC4, JDEC5, JDEC6, JDEC7, JDEC8, JDEC9: Conn_01x01, Connector_PinSocket_2.54mm:PinSocket_1x01_P2.54mm_Vertical, symbol Connector_Generic:Conn_01x01
- added R10, R11, R4, R5, R6, R7, R8, R9: 4.7k, kpm-jlcpcb-basic:R_0402_1005Metric, symbol kpm-jlcpcb-basic:4.7k R 0402
- added R12, R14: 100k, kpm-jlcpcb-basic:R_0402_1005Metric, symbol kpm-jlcpcb-basic:100k R 0402
- added R13: 1k, kpm-jlcpcb-basic:R_0603_1608Metric, symbol kpm-jlcpcb-basic:1k R 0603
- added R2, R3: 150k, kpm-jlcpcb-basic:R_0402_1005Metric, symbol kpm-jlcpcb-basic:150k R 0402
- added SW1, SW2, SW3, SW4, SW41, SW42, SW43, SW44, SW45, SW46, SW47, SW48, SW5, SW6, SW7, SW8: PUSHBTN_DPDT_LATCH, EuroRackTools:SMD switch 6pin, symbol EuroRackTools:PUSHBTN_DPDT_LATCH
- added U12: CD4017BM, EuroRackTools:SOP-16_4.4x10.4mm_P1.27mm, symbol EuroRackTools:CD4017
- J1: lcsc C383608 -> (none)
- renumbered J2 to JCLK1
Connections:
- net +12V: no longer U2.16 (VDD)
- net +5V: now also U2.16 (VDD), J10.5 (Pin_5), J12.5 (Pin_5), J14.5 (Pin_5), J16.5 (Pin_5), J18.5 (Pin_5), J20.5 (Pin_5), J6.5 (Pin_5), J8.5 (Pin_5), R2.1, SW1.5 (A), SW2.5 (A), SW3.5 (A), SW4.5 (A), SW5.5 (A), SW6.5 (A), SW7.5 (A), SW8.5 (A), U12.16 (VDD)
- net GND: now also J10.1 (Pin_1), J12.1 (Pin_1), J14.1 (Pin_1), J16.1 (Pin_1), J18.1 (Pin_1), J20.1 (Pin_1), J6.1 (Pin_1), J8.1 (Pin_1), JCLK2.S (GND), JDEC20.1 (Pin_1), JDEC21.1 (Pin_1), JOUT1.S (GND), R10.2, R11.2, R14.2, R3.2, R4.2, R5.2, R6.2, R7.2, R8.2, R9.2, U12.13 (CKEN), U12.8 (VSS)
- net clock: now also D17.1 (K), J3.1 (Pin_1), J4.1 (Pin_1); no longer U1.2 (-)
- net at U3.1: now also R12.1
- net at U4.5 (+): now also J22.2 (Pin_2)
- net at U4.6 (-): now also J22.1 (Pin_1)
- net at U4.7: now also JDEC19.1 (Pin_1)
- net at U3.6 (-): now also U3.7, R13.1
- net at U4.1: now also JDEC18.1 (Pin_1)
- net at U4.2 (-): now also J21.1 (Pin_1)
- net at U4.3 (+): now also J21.2 (Pin_2)
- net at U3.5 (+): now also D18.1 (K), R14.1
- net at U3.3 (+): now also D2.1 (K), D7.1 (K), D11.1 (K), D13.1 (K), D15.1 (K), D3.1 (K), D5.1 (K), D9.1 (K)
- net at D2.2 (A): now also SW1.3 (B)
- net at U1.3 (+): now also JCLK1.T; no longer JCLK1.TN
- net at D7.2 (A): now also SW4.3 (B)
- net at U2.15 (Reset): now also U2.9 (Q8)
- net ref: now reaches U3.2 (-)
- net ref: now also U1.2 (-), J4.2 (Pin_2)
- net at U1.5 (+): now also JDEC17.1 (Pin_1)
- net at U1.6 (-), U1.7: now also JCLK2.T
- net beat1: no longer names the net of U2.3 (Q0)
- net beat1: now also SW1.2 (A)
- net beat2: no longer names the net of U2.2 (Q1)
- net beat2: now also SW2.2 (A)
- net beat3: no longer names the net of U2.4 (Q2)
- net beat3: now also SW3.2 (A)
- net beat4: no longer names the net of U2.7 (Q3)
- net beat4: now also SW4.2 (A)
- net beat5: no longer names the net of U2.10 (Q4)
- net beat5: now also SW5.2 (A)
- net beat6: no longer names the net of U2.1 (Q5)
- net beat6: now also SW6.2 (A)
- net beat7: no longer names the net of U2.5 (Q6)
- net beat7: now also SW7.2 (A)
- net beat8: no longer names the net of U2.6 (Q7)
- net beat8: now also SW8.2 (A)
- new net: D3.2 (A), SW2.3 (B)
- new net: JDEC3.1 (Pin_1), U12.7 (Q3)
- new net: JDEC1.1 (Pin_1), U12.2 (Q1)
- new net: JOUT1.T, R13.2
- new net: R2.2, R3.1
- new net: D4.1 (K), R5.1
- new net: D14.1 (K), R10.1
- new net: D12.1 (K), R9.1
- new net: D12.2 (A), SW6.6 (B)
- new net: J14.2 (Pin_2), SW45.4 (A)
- new net: J14.3 (Pin_3), SW45.5 (A)
- new net: J14.4 (Pin_4), SW45.6 (B)
- new net: D10.1 (K), R8.1
- new net: D10.2 (A), SW5.6 (B)
- new net: J2.1 (Pin_1), U12.14 (CLK)
- new net: J4.3 (Pin_3), JDEC10.1 (Pin_1), JDEC11.1 (Pin_1), JDEC12.1 (Pin_1), JDEC13.1 (Pin_1), JDEC14.1 (Pin_1), JDEC15.1 (Pin_1), JDEC16.1 (Pin_1), JDEC9.1 (Pin_1)
- new net: D17.2 (A), D18.2 (A), R12.2
- new net: J18.2 (Pin_2), SW47.4 (A)
- new net: J18.3 (Pin_3), SW47.5 (A)
- new net: J18.4 (Pin_4), SW47.6 (B)
- new net: J6.2 (Pin_2), SW41.4 (A)
- new net: J6.3 (Pin_3), SW41.5 (A)
- new net: J6.4 (Pin_4), SW41.6 (B)
- new net: J5.1 (Pin_1), SW41.1 (A)
- new net: J5.2 (Pin_2), SW41.2 (A)
- new net: J5.3 (Pin_3), SW41.3 (B)
- new net: J11.1 (Pin_1), SW43.1 (A)
- new net: J11.2 (Pin_2), SW43.2 (A)
- new net: J11.3 (Pin_3), SW43.3 (B)
- new net: D9.2 (A), SW5.3 (B)
- new net: J7.1 (Pin_1), SW42.1 (A)
- new net: J7.2 (Pin_2), SW42.2 (A)
- new net: J7.3 (Pin_3), SW42.3 (B)
- new net: J8.2 (Pin_2), SW42.4 (A)
- new net: J8.3 (Pin_3), SW42.5 (A)
- new net: J8.4 (Pin_4), SW42.6 (B)
- new net: JDEC5.1 (Pin_1), U12.1 (Q5)
- new net: JDEC4.1 (Pin_1), U12.10 (Q4)
- new net: U12.15 (Reset), U12.9 (Q8)
- new net: JDEC8.1 (Pin_1), U12.3 (Q0)
- new net: JDEC2.1 (Pin_1), U12.4 (Q2)
- new net: JDEC6.1 (Pin_1), U12.5 (Q6)
- new net: JDEC7.1 (Pin_1), U12.6 (Q7)
- new net: D1.1 (K), R4.1
- new net: D14.2 (A), SW7.6 (B)
- new net: J10.2 (Pin_2), SW44.4 (A)
- new net: J10.3 (Pin_3), SW44.5 (A)
- new net: J10.4 (Pin_4), SW44.6 (B)
- new net: D8.1 (K), R7.1
- new net: D8.2 (A), SW4.6 (B)
- new net: D13.2 (A), SW7.3 (B)
- new net: J9.1 (Pin_1), SW44.1 (A)
- new net: J9.2 (Pin_2), SW44.2 (A)
- new net: J9.3 (Pin_3), SW44.3 (B)
- new net: J17.1 (Pin_1), SW47.1 (A)
- new net: J17.2 (Pin_2), SW47.2 (A)
- new net: J17.3 (Pin_3), SW47.3 (B)
- new net: D15.2 (A), SW8.3 (B)
- new net: D16.2 (A), SW8.6 (B)
- new net: D11.2 (A), SW6.3 (B)
- new net: D16.1 (K), R11.1
- new net: D5.2 (A), SW3.3 (B)
- new net: D6.2 (A), SW3.6 (B)
- new net: J12.2 (Pin_2), SW43.4 (A)
- new net: J12.3 (Pin_3), SW43.5 (A)
- new net: J12.4 (Pin_4), SW43.6 (B)
- new net: J20.2 (Pin_2), SW48.4 (A)
- new net: J20.3 (Pin_3), SW48.5 (A)
- new net: J20.4 (Pin_4), SW48.6 (B)
- new net: D1.2 (A), SW1.6 (B)
- new net: J16.2 (Pin_2), SW46.4 (A)
- new net: J16.3 (Pin_3), SW46.5 (A)
- new net: J16.4 (Pin_4), SW46.6 (B)
- new net: J13.1 (Pin_1), SW45.1 (A)
- new net: J13.2 (Pin_2), SW45.2 (A)
- new net: J13.3 (Pin_3), SW45.3 (B)
- new net: J15.1 (Pin_1), SW46.1 (A)
- new net: J15.2 (Pin_2), SW46.2 (A)
- new net: J15.3 (Pin_3), SW46.3 (B)
- new net: D6.1 (K), R6.1
- new net: J19.1 (Pin_1), SW48.1 (A)
- new net: J19.2 (Pin_2), SW48.2 (A)
- new net: J19.3 (Pin_3), SW48.3 (B)
- new net: D4.2 (A), SW2.6 (B)
Other:
- note added: "https://www.falstad.com/circuit/circuitjs.html?ctz=CQAgjCAMB0l3BWEA2aAWB8CcBmSy0AOBBAdkJE0pDR0oFMBaMMAKACVw00UetleUEACYQhSCOhJhUkDmhg0YBFmHIEOBISylcUBcIQcuPMMIr9w5oaPGTps+auRYskQmBeFSwpTxhmRpyKpqoglmBhErbRsjJIaNCkZjiE2uKpaC76gcYhIggCloYC0WKxDkgI6DrkybTkwmCpOYasAM4mgr4SBEISAGYAhgA27fQdXWYUPVYUEhDDYxOd+ZGis+v9IEvjk-klImjRhUKLo3sA7nLCvTw4t3NQrNcPC9Zv4MgSkC83C99-uAon9PltPodfpxDjgcAJbhRYaURLx3tsYIQ-sc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"
- moved on the sheet: J1, JCLK1, U2
